File: PCB Schematic/PCB_Robolime/PCB_Robolime.kicad_sch (KiCad schematic)
At the start: 0 parts

Commit message: Push
Parts:
- added +5V: Conn_01x02_Socket, Package_TO_SOT_SMD:TO-252-2, symbol Connector:Conn_01x02_Socket
- added A1: Arduino_Nano_v3.x, Module:Arduino_Nano, symbol MCU_Module:Arduino_Nano_v3.x
- added NEO6M: ZC323200, ZC323200:XCVR_ZC323200, symbol ZC323200:ZC323200
- added U1: (no value), ESP32_30pin, symbol esp32_30pin_revised:ESP32_30Pin
- added U2: Ai-Thinker-Ra-02, RF_Module:Ai-Thinker-Ra-01-LoRa, symbol RF_Module:Ai-Thinker-Ra-02
Connections:
- new net: +5V.2 (Pin_2), A1.30 (VIN), NEO6M.1 (VCC), U1.1 (VIN)
- new net: U1.16 (3.3v), U2.3 (VDD)
- new net: U1.19 (GPIO2), U2.5 (DIO0)
- new net: NEO6M.3 (TX), U1.21 (GPIO16)
- new net: NEO6M.2 (RX), U1.22 (GPIO17)
- new net: U1.23 (GPIO5), U2.15 (~{NSS})
- new net: U1.24 (GPIO18), U2.12 (SCK)
- new net: U1.25 (GPIO19), U2.13 (MISO)
- new net: U1.30 (GPIO23), U2.14 (MOSI)
- new net: U1.5 (GPIO14), U2.4 (~{RESET})
- new net: NEO6M.SH1 (SHIELD), NEO6M.SH2 (SHIELD), NEO6M.SH3 (SHIELD), NEO6M.SH4 (SHIELD)
- new net GND: +5V.1 (Pin_1), A1.29 (GND), A1.4 (GND), NEO6M.4 (GND), U1.17 (GND), U1.2 (GND), U2.1 (GND), U2.16 (GND), U2.2 (GND), U2.9 (GND)
